File: kicad/try1.kicad_pcb (KiCad board)
At the start: 2 copper layers, 101.6 x 100.3 mm, 115 parts, among them J1 Conn_02x12_Odd_Even, J2 Conn_01x08_Female, J3 Conn_01x03, J4 USB_A, J5 USB_B_Micro, SW1 LL3301NF065QG-proy, SW2 LL3301NF065QG-proy, U1 ICE40UP5K-SG48ITR50-proy, U10 ZLDO1117G33TA-proy, U2 AD7918BRUZ-proy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

Commit message: Add files via upload
Parts:
- J1: value Conn_02x12_Odd_Even -> Conn_02x11_Odd_Even; footprint Connector_PinHeader_2.54mm:PinHeader_2x12_P2.54mm_Vertical -> Connector_PinHeader_2.54mm:PinHeader_2x11_P2.54mm_Vertical
- U10, U6, U7, U8, U9: footprint Package_TO_SOT_SMD:SOT-223-3_TabPin2 -> Package_TO_SOT_SMD:SOT-223
- moved R11 315.2 mm to (119.1, 72.2)
- moved D1 301.0 mm to (95.8, 95.6), turned to 270 degrees
- moved R12 284.8 mm to (92.0, 83.8), turned to 90 degrees
- moved C24 271.8 mm to (94.9, 83.7), turned to 270 degrees
- moved C14 269.5 mm to (118.9, 74.0)
- moved SW1 265.1 mm to (117.2, 78.4), turned to 180 degrees
- moved C6 254.6 mm to (96.3, 98.7)
- moved C1 233.8 mm to (123.0, 143.3)
- moved C4 233.8 mm to (36.3, 154.0)
- moved C5 233.8 mm to (20.0, 158.4)
- moved C7 233.8 mm to (88.7, 142.5)
- moved R2 233.8 mm to (103.1, 140.4)
- moved C2 233.8 mm to (54.3, 156.5)
- moved C3 233.8 mm to (110.4, 137.9)
- moved C8 233.8 mm to (81.4, 140.0)
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Connections:
- J1 pad 10: /FPGA_ICE40UP5K/PIO14 -> /FPGA_ICE40UP5K/PIO10
- J1 pad 11: /FPGA_ICE40UP5K/PIO3 -> /FPGA_ICE40UP5K/PIO11
- J1 pad 12: /FPGA_ICE40UP5K/PIO15 -> /FPGA_ICE40UP5K/PIO12
- J1 pad 13: /FPGA_ICE40UP5K/PIO4 -> /FPGA_ICE40UP5K/PIO13
- J1 pad 14: /FPGA_ICE40UP5K/PIO16 -> /FPGA_ICE40UP5K/PIO14
- J1 pad 15: /FPGA_ICE40UP5K/PIO5 -> /FPGA_ICE40UP5K/PIO15
- J1 pad 16: /FPGA_ICE40UP5K/PIO17 -> /FPGA_ICE40UP5K/PIO16
- J1 pad 17: /FPGA_ICE40UP5K/PIO6 -> /FPGA_ICE40UP5K/PIO17
- J1 pad 19: /FPGA_ICE40UP5K/PIO7 -> /FPGA_ICE40UP5K/PIO19
- J1 pad 2: /FPGA_ICE40UP5K/PIO10 -> GND
- J1 pad 20: /FPGA_ICE40UP5K/PIO19 -> /FPGA_ICE40UP5K/PIO20
- J1 pad 21: /FPGA_ICE40UP5K/PIO8 -> /FPGA_ICE40UP5K/PIO21
- J1 pad 22: /FPGA_ICE40UP5K/PIO20 -> /FPGA_ICE40UP5K/PIO22
- J1 pad 3: +3.3V_FPGA -> /FPGA_ICE40UP5K/PIO3
- J1 pad 4: /FPGA_ICE40UP5K/PIO11 -> /FPGA_ICE40UP5K/PIO4
- J1 pad 5: GND -> /FPGA_ICE40UP5K/PIO5
- J1 pad 6: /FPGA_ICE40UP5K/PIO12 -> /FPGA_ICE40UP5K/PIO6
- J1 pad 7: /FPGA_ICE40UP5K/PIO1 -> /FPGA_ICE40UP5K/PIO7
- J1 pad 8: /FPGA_ICE40UP5K/PIO13 -> /FPGA_ICE40UP5K/PIO8
- J1 pad 9: /FPGA_ICE40UP5K/PIO2 -> /FPGA_ICE40UP5K/PIO9
- R18 pad 2: (no net) -> /FPGA_ICE40UP5K/ICE40_SDO
- R19 pad 2: (no net) -> /FPGA_ICE40UP5K/ICE40_SDI
- U1 pad 10: /FPGA_ICE40UP5K/PIO11 -> /FPGA_ICE40UP5K/PIO3
- U1 pad 11: /FPGA_ICE40UP5K/PIO12 -> /FPGA_ICE40UP5K/I2C_FPGA_SCL
- U1 pad 12: /FPGA_ICE40UP5K/PIO13 -> /FPGA_ICE40UP5K/I2C_FPGA_SDA
- U1 pad 13: /FPGA_ICE40UP5K/I2C_FPGA_SDA -> (no net)
- U1 pad 14: /FPGA_ICE40UP5K/ICE40_SDO -> (no net)
- U1 pad 15: /FPGA_ICE40UP5K/ICE40_SCK -> /FPGA_ICE40UP5K/ICE40_SDO
- U1 pad 18: /FPGA_ICE40UP5K/PIO16 -> /FPGA_ICE40UP5K/ICE40_CMISO
- U1 pad 19: /FPGA_ICE40UP5K/PIO15 -> /FPGA_ICE40UP5K/ICE40_CSCK
- U1 pad 2: /FPGA_ICE40UP5K/PIO6 -> /FPGA_ICE40UP5K/PIO8
- U1 pad 20: /FPGA_ICE40UP5K/PIO14 -> /FPGA_ICE40UP5K/CLK_IN
- U1 pad 21: /FPGA_ICE40UP5K/I2C_FPGA_SCL -> /FPGA_ICE40UP5K/ICE40_CMOSI
- U1 pad 23: /FPGA_ICE40UP5K/PIO18 -> /FPGA_ICE40UP5K/ICE40_CSS
- U1 pad 25: /FPGA_ICE40UP5K/PIO17 -> /FPGA_ICE40UP5K/ADC_SCLK
- U1 pad 26: /FPGA_ICE40UP5K/PIO20 -> /FPGA_ICE40UP5K/ADC_DIN
- U1 pad 27: /FPGA_ICE40UP5K/PIO19 -> /FPGA_ICE40UP5K/ADC_CS
- U1 pad 28: /FPGA_ICE40UP5K/PIO21 -> /FPGA_ICE40UP5K/ADC_DOUT
- U1 pad 3: /FPGA_ICE40UP5K/PIO8 -> /FPGA_ICE40UP5K/PIO7
- U1 pad 31: /FPGA_ICE40UP5K/ADC_CS -> /FPGA_ICE40UP5K/PIO22
- U1 pad 32: /FPGA_ICE40UP5K/ADC_DIN -> /FPGA_ICE40UP5K/PIO21
- U1 pad 34: /FPGA_ICE40UP5K/ADC_DOUT -> /FPGA_ICE40UP5K/PIO20
- U1 pad 35: /FPGA_ICE40UP5K/CLK_IN -> /FPGA_ICE40UP5K/PIO19
- U1 pad 36: /FPGA_ICE40UP5K/ICE40_CMISO -> /FPGA_ICE40UP5K/PIO18
- U1 pad 37: /FPGA_ICE40UP5K/ADC_SCLK -> /FPGA_ICE40UP5K/PIO17
- U1 pad 38: /FPGA_ICE40UP5K/ICE40_CMOSI -> /FPGA_ICE40UP5K/PIO16
- U1 pad 4: /FPGA_ICE40UP5K/PIO7 -> /FPGA_ICE40UP5K/PIO6
- U1 pad 42: /FPGA_ICE40UP5K/ICE40_CSS -> /FPGA_ICE40UP5K/PIO15
- U1 pad 43: /FPGA_ICE40UP5K/ICE40_CSCK -> /FPGA_ICE40UP5K/PIO14
- U1 pad 44: /FPGA_ICE40UP5K/PIO3 -> /FPGA_ICE40UP5K/PIO13
- U1 pad 45: /FPGA_ICE40UP5K/PIO5 -> /FPGA_ICE40UP5K/PIO12
- U1 pad 46: /FPGA_ICE40UP5K/PIO1 -> /FPGA_ICE40UP5K/PIO11
- U1 pad 47: /FPGA_ICE40UP5K/PIO2 -> /FPGA_ICE40UP5K/PIO10
- U1 pad 48: /FPGA_ICE40UP5K/PIO4 -> /FPGA_ICE40UP5K/PIO9
- U1 pad 6: /FPGA_ICE40UP5K/PIO9 -> /FPGA_ICE40UP5K/PIO5
- U1 pad 9: /FPGA_ICE40UP5K/PIO10 -> /FPGA_ICE40UP5K/PIO4
Routing:
- net /FPGA_ICE40UP5K/I2C_FPGA_SCL: track 0.00 -> 52.4 mm, vias 0 -> 1
- net /FPGA_ICE40UP5K/I2C_FPGA_SDA: track 0.00 -> 46.2 mm, vias 0 -> 1
- net /FPGA_ICE40UP5K/ICE40_SS: track 0.00 -> 39.9 mm
- net /FPGA_ICE40UP5K/ICE40_SCK: track 0.00 -> 31.3 mm, vias 0 -> 2
- net /FPGA_ICE40UP5K/CRESET_B: track 0.00 -> 31.1 mm, vias 0 -> 2
- net /FPGA_ICE40UP5K/ICE40_SDI: track 0.00 -> 29.8 mm, vias 0 -> 2
- net /FPGA_ICE40UP5K/PIO22: track 0.00 -> 29.4 mm
- net /FPGA_ICE40UP5K/PIO20: track 0.00 -> 26.1 mm
- net /FPGA_ICE40UP5K/PIO21: track 0.00 -> 25.1 mm
- net /FPGA_ICE40UP5K/PIO18: track 0.00 -> 23.0 mm
- net /FPGA_ICE40UP5K/PIO4: track 0.00 -> 21.5 mm
- net /FPGA_ICE40UP5K/PIO19: track 0.00 -> 21.3 mm
- net /FPGA_ICE40UP5K/PIO16: track 0.00 -> 20.9 mm
- net /FPGA_ICE40UP5K/PIO14: track 0.00 -> 20.2 mm
- net /FPGA_ICE40UP5K/ADC_CS: track 0.00 -> 19.3 mm
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Other:
- board size 101.6 x 100.3 mm -> 100.3 x 100.3 mm
- rule via_min_drill: 0.3 -> 0.1
- rule via_min_size: 0.4 -> 0.2

Commit message: Add files via upload
Parts:
- removed C6: 0.1uF, Resistor_SMD:R_0603_1608Metric_Pad1.05x0.95mm_HandSolder
- removed D1: 1N5819, Diode_SMD:D_SOD-123
- C14, C34, C36: footprint Resistor_SMD:R_0805_2012Metric_Pad1.15x1.40mm_HandSolder -> Resistor_SMD:R_0603_1608Metric_Pad1.05x0.95mm_HandSolder
- D2, D5: footprint LED_SMD:LED_0805_2012Metric_Pad1.15x1.40mm_HandSolder -> LED_SMD:LED_0603_1608Metric_Pad1.05x0.95mm_HandSolder
- SW1, SW2: footprint libreria_proyecto_fp:LL3301NF065QG -> libreria_proyecto_fp:LL3301NF065QG-proy
- moved FB7 109.3 mm to (75.4, 102.5), turned to 90 degrees
- moved C2 107.5 mm to (102.0, 60.2), turned to 270 degrees
- moved C30 102.4 mm to (76.9, 102.4), turned to 270 degrees
- moved C29 98.6 mm to (78.5, 102.4), turned to 270 degrees
- moved R15 96.8 mm to (81.7, 102.5), turned to 90 degrees
- moved C5 95.5 mm to (81.5, 85.3), turned to 90 degrees
- moved R16 94.8 mm to (67.5, 95.5), turned to 270 degrees
- moved C26 94.3 mm to (72.2, 102.5), turned to 270 degrees
- moved R17 93.0 mm to (80.1, 102.4), turned to 90 degrees
- moved C28 92.7 mm to (69.0, 102.5), turned to 270 degrees
- moved C25 88.4 mm to (73.8, 102.5), turned to 270 degrees
- moved R23 87.4 mm to (61.2, 54.6), turned to 270 degrees
- moved C27 87.1 mm to (70.6, 102.5), turned to 270 degrees
- moved C1 85.3 mm to (103.6, 60.2), turned to 270 degrees
- moved C4 83.1 mm to (83.1, 85.3), turned to 90 degrees
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Connections:
- net /FPGA_ICE40UP5K/ICE40_SDI renamed /FPGA_ICE40UP5K/ICE40_MOSI
- C31 pad 2: 3.3V_FPGA -> +3.3V_FPGA
- C7 pad 2: 3.3V_FPGA -> +3.3V_FPGA
- C8 pad 2: 3.3V_FPGA -> +3.3V_FPGA
- C9 pad 2: 3.3V_FPGA -> +3.3V_FPGA
- R13 pad 2: /FPGA_ICE40UP5K/ICE40_SS -> /FPGA_ICE40UP5K/ICE40_CS
- R18 pad 2: /FPGA_ICE40UP5K/ICE40_SDO -> /FPGA_ICE40UP5K/ICE40_MISO
- R2 pad 1: 3.3V_FPGA -> +3.3V_FPGA
- R20 pad 2: /FPGA_ICE40UP5K/ICE40_SS -> /FPGA_ICE40UP5K/ICE40_CLK
- R21 pad 2: /FPGA_ICE40UP5K/ICE40_SCK -> /FPGA_ICE40UP5K/ICE40_CS
- U1 pad 1: 3.3V_FPGA -> +3.3V_FPGA
- U1 pad 10: /FPGA_ICE40UP5K/PIO3 -> /FPGA_ICE40UP5K/PIO4
- U1 pad 14: (no net) -> /FPGA_ICE40UP5K/ICE40_MISO
- U1 pad 15: /FPGA_ICE40UP5K/ICE40_SDO -> /FPGA_ICE40UP5K/ICE40_CLK
- U1 pad 16: /FPGA_ICE40UP5K/ICE40_SS -> /FPGA_ICE40UP5K/ICE40_CS
- U1 pad 18: /FPGA_ICE40UP5K/ICE40_CMISO -> /FPGA_ICE40UP5K/ICE40_CMOSI
- U1 pad 19: /FPGA_ICE40UP5K/ICE40_CSCK -> /FPGA_ICE40UP5K/ICE40_CMISO
- U1 pad 2: /FPGA_ICE40UP5K/PIO8 -> /FPGA_ICE40UP5K/PIO7
- U1 pad 21: /FPGA_ICE40UP5K/ICE40_CMOSI -> /FPGA_ICE40UP5K/ICE40_CSCK
- U1 pad 22: 3.3V_FPGA -> +3.3V_FPGA
- U1 pad 24: Net-(D1-Pad1) -> +2.5V_FPGA
- U1 pad 3: /FPGA_ICE40UP5K/PIO7 -> /FPGA_ICE40UP5K/PIO8
- U1 pad 31: /FPGA_ICE40UP5K/PIO22 -> /FPGA_ICE40UP5K/PIO21
- U1 pad 32: /FPGA_ICE40UP5K/PIO21 -> /FPGA_ICE40UP5K/PIO22
- U1 pad 33: 3.3V_FPGA -> +3.3V_FPGA
- U1 pad 34: /FPGA_ICE40UP5K/PIO20 -> /FPGA_ICE40UP5K/PIO19
- U1 pad 35: /FPGA_ICE40UP5K/PIO19 -> /FPGA_ICE40UP5K/PIO20
- U1 pad 36: /FPGA_ICE40UP5K/PIO18 -> /FPGA_ICE40UP5K/PIO17
- U1 pad 37: /FPGA_ICE40UP5K/PIO17 -> /FPGA_ICE40UP5K/PIO18
- U1 pad 38: /FPGA_ICE40UP5K/PIO16 -> /FPGA_ICE40UP5K/PIO15
- U1 pad 4: /FPGA_ICE40UP5K/PIO6 -> /FPGA_ICE40UP5K/PIO5
- U1 pad 42: /FPGA_ICE40UP5K/PIO15 -> /FPGA_ICE40UP5K/PIO16
- U1 pad 43: /FPGA_ICE40UP5K/PIO14 -> /FPGA_ICE40UP5K/PIO13
- U1 pad 44: /FPGA_ICE40UP5K/PIO13 -> /FPGA_ICE40UP5K/PIO14
- U1 pad 45: /FPGA_ICE40UP5K/PIO12 -> /FPGA_ICE40UP5K/PIO11
- U1 pad 46: /FPGA_ICE40UP5K/PIO11 -> /FPGA_ICE40UP5K/PIO12
- U1 pad 47: /FPGA_ICE40UP5K/PIO10 -> /FPGA_ICE40UP5K/PIO9
- U1 pad 48: /FPGA_ICE40UP5K/PIO9 -> /FPGA_ICE40UP5K/PIO10
- U1 pad 6: /FPGA_ICE40UP5K/PIO5 -> /FPGA_ICE40UP5K/PIO6
- U1 pad 9: /FPGA_ICE40UP5K/PIO4 -> /FPGA_ICE40UP5K/PIO3
- U3 pad 1: /FPGA_ICE40UP5K/ICE40_SS -> /FPGA_ICE40UP5K/ICE40_CS
- U3 pad 5: /FPGA_ICE40UP5K/ICE40_SDO -> /FPGA_ICE40UP5K/ICE40_MISO
- U3 pad 6: /FPGA_ICE40UP5K/ICE40_SCK -> /FPGA_ICE40UP5K/ICE40_CLK
- U4 pad 20: /FPGA_ICE40UP5K/ICE40_CMISO -> /FPGA_ICE40UP5K/ICE40_CSS
- U4 pad 22: /FPGA_ICE40UP5K/ICE40_CMOSI -> /FPGA_ICE40UP5K/ICE40_CMISO
- U4 pad 23: /FPGA_ICE40UP5K/ICE40_CSS -> /FPGA_ICE40UP5K/ICE40_CMOSI
- U4 pad 42: /Onion_2/UART_RX -> (no net)
- U4 pad 43: /STM_32/UART_RX -> (no net)
- U4 pad 51: (no net) -> /STM_32/UART_M_TX
- U4 pad 52: (no net) -> /STM_32/UART_M_RX
- U5 pad 8: /Onion_2/UART_RX -> /STM_32/UART_M_TX
- U5 pad 9: /STM_32/UART_RX -> /STM_32/UART_M_RX
Routing:
- net GND: track 4.50 -> 339.8 mm, vias 0 -> 20
- net +5V: track 8.65 -> 252.6 mm, vias 0 -> 3
- net +3.3V_FPGA: track 3.28 -> 128.6 mm, vias 0 -> 10
- net +3.3V_micro: track 0.00 -> 100.1 mm, vias 0 -> 7
- net +3.3V_omega: track 0.00 -> 87.2 mm, vias 0 -> 2
- net /Onion_2/BOOT1: track 0.00 -> 82.4 mm
- net +1.2V_FPGA: track 0.00 -> 73.0 mm, vias 0 -> 5
- net /FPGA_ICE40UP5K/I2C_FPGA_SDA: track 46.2 -> 115.9 mm
- net /FPGA_ICE40UP5K/I2C_FPGA_SCL: track 52.4 -> 114.4 mm, vias 1 -> 0
- net +2.5V_FPGA: track 3.47 -> 57.0 mm, vias 0 -> 4
- net /Onion_2/RST: track 0.00 -> 53.1 mm, vias 0 -> 1
- net /Onion_2/BOOT0: track 0.00 -> 47.1 mm, vias 0 -> 1
- net /FPGA_ICE40UP5K/ICE40_SS: track 39.9 -> 0.00 mm
- net /FPGA_ICE40UP5K/ICE40_CLK: track 0.00 -> 38.9 mm, vias 0 -> 3
- net /Onion_2/USB_D-: track 0.00 -> 38.0 mm, vias 0 -> 2
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- added copper zone on F.Cu, net GND
Other:
- board size 100.3 x 100.3 mm -> 83.8 x 68.6 mm
- rule via_min_size: 0.2 -> 0.4

Commit message: Add files via upload
Parts:
- moved SW2 2.63 mm to (66.7, 47.2), turned to 180 degrees
- moved J1 2.39 mm to (111.4, 74.0)
- moved FB6 0.95 mm to (108.6, 107.0)
- moved FB4 0.76 mm to (42.1, 108.0)
Routing:
- net GND: track 339.8 -> 224.2 mm, vias 20 -> 13
- net +5V: track 252.6 -> 194.3 mm
- net +3.3V_FPGA: track 128.6 -> 136.6 mm
- net /FPGA_ICE40UP5K/PIO13: track 19.0 -> 15.4 mm
- net /FPGA_ICE40UP5K/PIO14: track 21.6 -> 18.0 mm
- net /FPGA_ICE40UP5K/PIO16: track 22.9 -> 19.5 mm
- net /FPGA_ICE40UP5K/PIO15: track 18.3 -> 15.4 mm
- net /FPGA_ICE40UP5K/PIO21: track 25.2 -> 22.4 mm
- net /Onion_2/RST: track 53.1 -> 55.9 mm
- net /FPGA_ICE40UP5K/PIO5: track 17.6 -> 14.9 mm
- net /FPGA_ICE40UP5K/PIO10: track 17.9 -> 15.3 mm
- net /FPGA_ICE40UP5K/PIO9: track 15.1 -> 12.6 mm
- net /FPGA_ICE40UP5K/PIO11: track 16.7 -> 14.3 mm
- net /FPGA_ICE40UP5K/PIO22: track 26.6 -> 24.3 mm
- net /FPGA_ICE40UP5K/PIO3: track 20.8 -> 18.5 mm
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- added copper zone on B.Cu, net GND

Commit message: Add files via upload
Routing:
- net +2.5V_FPGA: track 57.4 -> 63.9 mm
- net GND: track 224.2 -> 222.2 mm, vias 13 -> 14
- net +5V: track 194.3 -> 195.7 mm
- net /FPGA_ICE40UP5K/I2C_FPGA_SCL: track 114.4 -> 113.7 mm

Commit message: Add files via upload
Parts:
- moved R14 1.31 mm to (79.7, 74.0)
- moved C23 0.28 mm to (90.0, 91.8)
- moved C22 0.25 mm to (90.0, 90.1)
Routing:
- net GND: track 222.2 -> 6.09 mm, vias 14 -> 194
- net /FPGA_ICE40UP5K/ICE40_MOSI: track 37.2 -> 42.3 mm
- net +2.5V_FPGA: track 63.9 -> 67.4 mm
- net /FPGA_ICE40UP5K/ICE40_CS: track 35.5 -> 38.3 mm
- net +3.3V_FPGA: track 136.6 -> 139.2 mm
- net /FPGA_ICE40UP5K/ADC_CS: track 11.5 -> 13.3 mm
- net Net-(C12-Pad2): track 13.6 -> 15.4 mm
- net /FPGA_ICE40UP5K/ADC_DIN: track 10.6 -> 12.3 mm
- net +3.3V_micro: track 102.3 -> 103.8 mm
- net Net-(C15-Pad2): track 10.6 -> 12.0 mm
- net Net-(C13-Pad2): track 12.5 -> 13.7 mm
- net Net-(R14-Pad1): track 1.85 -> 3.07 mm
- net Net-(C10-Pad2): track 14.8 -> 13.7 mm
- net /Onion_2/RST: track 55.9 -> 54.8 mm
- net Net-(C4-Pad2): track 20.8 -> 19.8 mm
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