File: kicad/try1.kicad_pcb (KiCad board)
At the start: 2 copper layers, 83.8 x 68.6 mm, 113 parts, among them J1 Conn_02x11_Odd_Even, J2 Conn_01x08_Female, J3 Conn_01x03, J4 USB_A, J5 USB_B_Micro, SW1 LL3301NF065QG-proy, SW2 LL3301NF065QG-proy, U1 ICE40UP5K-SG48ITR50-proy, U10 ZLDO1117G33TA-proy, U2 AD7918BRUZ-proy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

Commit message: Add files via upload
Parts:
- added FB10: BLM18SG121TN1D-proy, Resistor_SMD:R_0603_1608Metric_Pad1.05x0.95mm_HandSolder, F.Cu at (40.0, 52.0)
- added FB8: BLM18SG121TN1D-proy, Resistor_SMD:R_0603_1608Metric_Pad1.05x0.95mm_HandSolder, F.Cu at (67.5, 106.6)
- added FB9: BLM18SG121TN1D-proy, Resistor_SMD:R_0603_1608Metric_Pad1.05x0.95mm_HandSolder, F.Cu at (110.0, 53.6)
- moved C32 2.36 mm to (64.9, 105.5), turned to 90 degrees
- moved C33 2.35 mm to (63.4, 105.5), turned to 90 degrees
- moved C49 0.35 mm to (81.6, 54.1)
- moved U9 0.27 mm to (77.8, 47.6)
Connections:
- J4 pad 5: GND -> Net-(FB10-Pad2)
- J5 pad 2: (no net) -> Net-(J5-Pad2)
- J5 pad 3: (no net) -> Net-(J5-Pad3)
- J5 pad 4: (no net) -> Net-(J5-Pad4)
- J5 pad 6: GND -> GND_case
- U1 pad 13: (no net) -> Net-(U1-Pad13)
- U1 pad 39: (no net) -> Net-(U1-Pad39)
- U1 pad 40: (no net) -> Net-(U1-Pad40)
- U1 pad 41: (no net) -> Net-(U1-Pad41)
- U4 pad 1: (no net) -> Net-(U4-Pad1)
- U4 pad 10: (no net) -> Net-(U4-Pad10)
- U4 pad 11: (no net) -> Net-(U4-Pad11)
- U4 pad 12: GND -> Net-(FB8-Pad2)
- U4 pad 14: (no net) -> Net-(U4-Pad14)
- U4 pad 15: (no net) -> Net-(U4-Pad15)
- U4 pad 16: (no net) -> Net-(U4-Pad16)
- U4 pad 17: (no net) -> Net-(U4-Pad17)
- U4 pad 2: (no net) -> Net-(U4-Pad2)
- U4 pad 24: (no net) -> Net-(U4-Pad24)
- U4 pad 25: (no net) -> Net-(U4-Pad25)
- U4 pad 26: (no net) -> Net-(U4-Pad26)
- U4 pad 27: (no net) -> Net-(U4-Pad27)
- U4 pad 29: (no net) -> Net-(U4-Pad29)
- U4 pad 3: (no net) -> Net-(U4-Pad3)
- U4 pad 30: (no net) -> Net-(U4-Pad30)
- U4 pad 33: (no net) -> Net-(U4-Pad33)
- U4 pad 34: (no net) -> Net-(U4-Pad34)
- U4 pad 35: (no net) -> Net-(U4-Pad35)
- U4 pad 36: (no net) -> Net-(U4-Pad36)
- U4 pad 37: (no net) -> Net-(U4-Pad37)
- U4 pad 38: (no net) -> Net-(U4-Pad38)
- U4 pad 39: (no net) -> Net-(U4-Pad39)
- U4 pad 4: (no net) -> Net-(U4-Pad4)
- U4 pad 40: (no net) -> Net-(U4-Pad40)
- U4 pad 41: (no net) -> Net-(U4-Pad41)
- U4 pad 42: (no net) -> Net-(U4-Pad42)
- U4 pad 43: (no net) -> Net-(U4-Pad43)
- U4 pad 44: (no net) -> Net-(U4-Pad44)
- U4 pad 45: (no net) -> Net-(U4-Pad45)
- U4 pad 5: (no net) -> Net-(U4-Pad5)
- U4 pad 53: (no net) -> Net-(U4-Pad53)
- U4 pad 54: (no net) -> Net-(U4-Pad54)
- U4 pad 57: (no net) -> Net-(U4-Pad57)
- U4 pad 6: (no net) -> Net-(U4-Pad6)
- U4 pad 61: (no net) -> Net-(U4-Pad61)
- U4 pad 62: (no net) -> Net-(U4-Pad62)
- U4 pad 7: (no net) -> Net-(U4-Pad7)
- U4 pad 8: (no net) -> Net-(U4-Pad8)
- U4 pad 9: (no net) -> Net-(U4-Pad9)
- U5 pad 16: (no net) -> Net-(U5-Pad16)
- U5 pad 20: (no net) -> Net-(U5-Pad20)
- U5 pad 21: (no net) -> Net-(U5-Pad21)
- U5 pad 22: (no net) -> Net-(U5-Pad22)
- U5 pad 23: (no net) -> Net-(U5-Pad23)
- U5 pad 24: (no net) -> Net-(U5-Pad24)
- U5 pad 25: (no net) -> Net-(U5-Pad25)
- U5 pad 7: (no net) -> Net-(U5-Pad7)
Routing:
- net GND_case: track 0.00 -> 23.0 mm, vias 0 -> 1
- net Net-(FB10-Pad2): track 0.00 -> 16.7 mm
- net Net-(FB8-Pad2): track 0.00 -> 14.2 mm, vias 0 -> 2
- net +2.5V_FPGA: track 67.4 -> 57.1 mm
- net /FPGA_ICE40UP5K/I2C_FPGA_SDA: track 118.0 -> 112.0 mm, vias 1 -> 5
- net Net-(C34-Pad1): track 23.8 -> 18.9 mm, vias 0 -> 2
- net +1.2V_FPGA: track 75.1 -> 70.2 mm
- net /FPGA_ICE40UP5K/I2C_FPGA_SCL: track 113.9 -> 109.4 mm, vias 0 -> 4
- net +3.3V_omega: track 86.8 -> 91.0 mm
- net +5V: track 196.3 -> 199.4 mm
- net Net-(D4-Pad2): track 12.1 -> 10.6 mm
- net /Onion_2/BOOT1: track 82.4 -> 83.9 mm, vias 0 -> 2
- net GND: track 6.09 -> 5.22 mm, vias 194 -> 324
- net Net-(C4-Pad2): track 19.8 -> 19.1 mm
- net +3.3V_micro: track 103.8 -> 104.4 mm
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Other:
- board text added: "DESIGNED BY: HAIR SEBASTIAN LOPEZ CRIOLLO"
