File: kicad/FPGA_ICE40UP5K.sch (KiCad schematic (older format))
At the start: 49 parts, among them J1 Conn_01x23_Female, J2 Conn_01x08_Female, SW1 LL3301NF065QG-proy, U1 ICE40UP5K-SG48ITR50-proy, U2 AD7918BRUZ-proy, U3 W25Q32JVSS-proy, X1 CWX823-025.0M-proy

Commit message: Remove duplicated directory
Parts:
- removed J1: Conn_01x23_Female, symbol Connector:Conn_01x23_Female
- added C31: 0.1uF, Resistor_SMD:R_0603_1608Metric_Pad1.05x0.95mm_HandSolder, symbol Device:C
- added J1: Conn_02x12_Odd_Even, Connector_PinHeader_2.54mm:PinHeader_2x12_P2.54mm_Vertical, symbol Connector_Generic:Conn_02x12_Odd_Even
- C1, C10, C11, C12, C13, C15, C16, C17, C18, C19, C2, C20, C21, C22, C23, C24, C3, C4, C5, C55, C6, C7, C8, C9: footprint Capacitor_SMD:C_0805_2012Metric_Pad1.15x1.40mm_HandSolder -> Resistor_SMD:R_0603_1608Metric_Pad1.05x0.95mm_HandSolder
- C14: footprint Capacitor_SMD:C_1206_3216Metric_Pad1.42x1.75mm_HandSolder -> Resistor_SMD:R_0805_2012Metric_Pad1.15x1.40mm_HandSolder
- J2: footprint (none) -> Connector_PinHeader_2.54mm:PinHeader_1x08_P2.54mm_Vertical
- R1, R10, R11, R12, R13, R14, R2, R25, R3, R4, R5, R6, R7, R8, R9: footprint Resistor_SMD:R_0805_2012Metric_Pad1.15x1.40mm_HandSolder -> Resistor_SMD:R_0603_1608Metric_Pad1.05x0.95mm_HandSolder
Connections:
- net labels added: +1.2V_FPGA, I2C_FPGA_SCL, I2C_FPGA_SDA, I2C_all0, I2C_all1, I2C_all[1..0], SPI_fo0, SPI_fo1, SPI_fo2, SPI_fo3, SPI_fo4, SPI_fo[4..0], SPI_mf0, SPI_mf1, SPI_mf2, SPI_mf3, SPI_mf[3..0]
- net labels removed: 1.2V_FPGA, I2C_F0, I2C_F1, I2C_SCL, I2C_SDA, I2C_fpga[1..0], RST, SPI_fpga0, SPI_fpga1, SPI_fpga2, SPI_fpga3, SPI_fpga4, SPI_fpga[3..0], SPI_fpga_omega[4..0]
- wire segments 175 -> 177

Commit message: Add files via upload
Parts:
- removed J1: Conn_02x12_Odd_Even, Connector_PinHeader_2.54mm:PinHeader_2x12_P2.54mm_Vertical, symbol Connector_Generic:Conn_02x12_Odd_Even
- added J1: Conn_02x11_Odd_Even, Connector_PinHeader_2.54mm:PinHeader_2x11_P2.54mm_Vertical, symbol Connector_Generic:Conn_02x11_Odd_Even
Connections:
- net labels added: PIO22
- net labels removed: ICE40_SD0, ICE40_SD1, PIO1, PIO2
- wire segments 177 -> 175
- no-connect marks 3 -> 4

Commit message: Add files via upload
Parts:
- removed C6: 0.1uF, Resistor_SMD:R_0603_1608Metric_Pad1.05x0.95mm_HandSolder, symbol Device:C
- removed D1: 1N5819, Diode_SMD:D_SOD-123, symbol Diode:1N5819
- C14: footprint Resistor_SMD:R_0805_2012Metric_Pad1.15x1.40mm_HandSolder -> Resistor_SMD:R_0603_1608Metric_Pad1.05x0.95mm_HandSolder
- D2: footprint LED_SMD:LED_0805_2012Metric_Pad1.15x1.40mm_HandSolder -> LED_SMD:LED_0603_1608Metric_Pad1.05x0.95mm_HandSolder
- SW1: footprint libreria_proyecto_fp:LL3301NF065QG -> libreria_proyecto_fp:LL3301NF065QG-proy
Connections:
- net 3.3V_FPGA is gone; now on net +3.3V_FPGA: C31.2, C7.2, C8.2, C9.2, R2.1, U1.1 (VCCIO_2), U1.22 (SPI_VCCIO1), U1.33 (VCCIO_0)
- net +2.5V_FPGA: now also U1.24 (VPP_2V5)
- net ICE40_CMISO: now also U1.19 (IOB_29B); no longer U1.18 (IOB_31B)
- net ICE40_CMOSI: now also U1.18 (IOB_31B); no longer U1.21 (IOB_23B)
- net ICE40_CSCK: now also U1.21 (IOB_23B); no longer U1.19 (IOB_29B)
- net PIO10: now also U1.48 (IOB_4A); no longer U1.47 (IOB_2A)
- net PIO11: now also U1.45 (IOB_5B); no longer U1.46 (IOB_0A)
- net PIO12: now also U1.46 (IOB_0A); no longer U1.45 (IOB_5B)
- net PIO13: now also U1.43 (IOT_49A); no longer U1.44 (IOT_3B_G6)
- net PIO14: now also U1.44 (IOT_3B_G6); no longer U1.43 (IOT_49A)
- net PIO15: now also U1.38 (IOT_50b); no longer U1.42 (IOT_51A)
- net PIO16: now also U1.42 (IOT_51A); no longer U1.38 (IOT_50b)
- net PIO17: now also U1.36 (IOT_48b); no longer U1.37 (IOT_45a_G1)
- net PIO18: now also U1.37 (IOT_45a_G1); no longer U1.36 (IOT_48b)
- net PIO19: now also U1.34 (IOT_44b); no longer U1.35 (IOT_46b_G0)
- net PIO20: now also U1.35 (IOT_46b_G0); no longer U1.34 (IOT_44b)
- net PIO21: now also U1.31 (IOT_42b); no longer U1.32 (IOT_43a)
- net PIO22: now also U1.32 (IOT_43a); no longer U1.31 (IOT_42b)
- net PIO3: now also U1.9 (IOB_16A); no longer U1.10 (IOB_18A)
- net PIO4: now also U1.10 (IOB_18A); no longer U1.9 (IOB_16A)
- net PIO5: now also U1.4 (IOB_8A); no longer U1.6 (IOB_13B)
- net PIO6: now also U1.6 (IOB_13B); no longer U1.4 (IOB_8A)
- net PIO7: now also U1.2 (IOB_6A); no longer U1.3 (IOB_9B)
- net PIO8: now also U1.3 (IOB_9B); no longer U1.2 (IOB_6A)
- net PIO9: now also U1.47 (IOB_2A); no longer U1.48 (IOB_4A)
- net ICE40_MISO: now reaches U1.14 (IOB_32A_SPI_SDO)
- net ICE40_MISO: now also U3.5 (DI(IO0))
- net ICE40_SCK renamed ICE40_CLK
- net ICE40_CLK: now also U1.15 (IOB_34A_SPI_SCK)
- net ICE40_SDI renamed ICE40_MOSI
- removed net ICE40_SDO: U1.15 (IOB_34A_SPI_SCK), U3.5 (DI(IO0))
- net ICE40_SS renamed ICE40_CS
- no-connect marks 4 -> 3
Other:
- moved on the sheet: J1

Commit message: Add files via upload
Parts:
- SW1: symbol proyecto_libreria:LL3301NF065QG-proy -> try1-rescue:LL3301NF065QG-proy-proyecto_libreria
- U1: symbol FPGA_Lattice:ICE40UP5K-SG48ITR50-proy -> try1-rescue:ICE40UP5K-SG48ITR50-proy-FPGA_Lattice
- U2: symbol Analog_ADC:AD7918BRUZ-proy -> try1-rescue:AD7918BRUZ-proy-Analog_ADC
- U3: symbol Memory_Flash:W25Q32JVSS-proy -> try1-rescue:W25Q32JVSS-proy-Memory_Flash
- X1: symbol Oscillator:CWX823-025.0M-proy -> try1-rescue:CWX823-025.0M-proy-Oscillator
Changed lines of the file:
@@
 $Descr User 14173 11811
 encoding utf-8
-Sheet 4 5
+Sheet 3 5
 Title ""
 Date ""
@@
 Connection ~ 3750 3000
 $Comp
-L Memory_Flash:W25Q32JVSS-proy U3
+L try1-rescue:W25Q32JVSS-proy-Memory_Flash U3
 U 1 1 5EDE2691
 P 11600 5850
@@
 Connection ~ 11600 6300
 $Comp
-L Analog_ADC:AD7918BRUZ-proy U2
+L try1-rescue:AD7918BRUZ-proy-Analog_ADC U2
 U 1 1 5EE2D889
 P 11700 2650
+AR Path="/5EE2D889" Ref="U2"  Part="1"
+AR Path="/5E81C2A4/5EE2D889" Ref="U2"  Part="1"
 F 0 "U2" V 11100 3000 60  0000 L CNN
 F 1 "AD7918BRUZ-proy" V 11200 2900 60  0000 L CNN
@@
 	7000 6050 10300 6050
 $Comp
-L Oscillator:CWX823-025.0M-proy X1
+L try1-rescue:CWX823-025.0M-proy-Oscillator X1
 U 1 1 5EB6DA64
 P 8850 6850
@@
 $EndComp
 $Comp
-L FPGA_Lattice:ICE40UP5K-SG48ITR50-proy U1
+L try1-rescue:ICE40UP5K-SG48ITR50-proy-FPGA_Lattice U1
 U 1 1 5EDC42AA
 P 2650 4150
@@
 $EndComp
 $Comp
-L proyecto_libreria:LL3301NF065QG-proy SW?
+L try1-rescue:LL3301NF065QG-proy-proyecto_libreria SW?
 U 1 1 5EBF33FF
 P 8450 5350
