File: kicad/Onion_2.sch (KiCad schematic (older format))
At the start: 19 parts, among them J3 Conn_01x03, J4 USB_A, SW2 LL3301NF065QG-proy, U5 Omega2+

Commit message: Remove duplicated directory
Parts:
- removed D3: BZX384C5V6-E3-08, Diode_SMD:D_SOD-323, symbol try1-rescue:BZX384C5V6-E3-08-BZX384C5V6-E3-08
- removed FerriteBead2: 742792651-proy, Inductor_SMD:L_0603_1608Metric_Pad1.05x0.95mm_HandSolder, symbol try1-rescue:742792651-proy-742792651
- removed U5: Omega2+, Module:Onion_Omega2+, symbol MCU_Module:Omega2+
- added D3: BZX384C5V6-E3-08-proy, libreria_proyecto_fp:SOD-323-proy, symbol Diode:BZX384C5V6-E3-08-proy
- added FB1: BLM18SG121TN1D-proy, Resistor_SMD:R_0603_1608Metric_Pad1.05x0.95mm_HandSolder, symbol proyecto_libreria:BLM18SG121TN1D-proy
- added U5: Omega2-proy, Module:Onion_Omega2+, symbol proyecto_libreria:Omega2-proy
- C32, C33, C35: footprint Capacitor_SMD:C_0805_2012Metric_Pad1.15x1.40mm_HandSolder -> Resistor_SMD:R_0603_1608Metric_Pad1.05x0.95mm_HandSolder
- C34, C36: footprint Capacitor_SMD:C_1206_3216Metric_Pad1.42x1.75mm_HandSolder -> Resistor_SMD:R_0805_2012Metric_Pad1.15x1.40mm_HandSolder
- J3: footprint (none) -> Connector_PinHeader_2.54mm:PinHeader_1x03_P2.54mm_Vertical
- R18, R19, R20, R21, R22, R23: footprint Resistor_SMD:R_0805_2012Metric_Pad1.15x1.40mm_HandSolder -> Resistor_SMD:R_0603_1608Metric_Pad1.05x0.95mm_HandSolder
Connections:
- net labels added: I2C_all0, I2C_all1, I2C_all[1..0], JTAG[4..0], SPI_MISO, SPI_MOSI, SPI_RST, SPI_fo0, SPI_fo1, SPI_fo2, SPI_fo3, SPI_fo4, SPI_fo[4..0]
- net labels removed: I2C_00, I2C_01, I2C_omega[1..0], JTAG5, JTAG[5..0], MISO, MOSI, NRST, OM_SPI0, OM_SPI1, OM_SPI2, OM_SPI3, OM_SPI4, RST_BTN, SPI_omega_fpga[4..0]
- wire segments 95 -> 92
- no-connect marks 6 -> 8

Commit message: Add files via upload
Changed lines of the file:
@@
 Wire Notes Line
 	8300 2650 5000 2650
-Wire Notes Line
-	600  550  8300 550
 Text Notes 6650 2450 0    118  ~ 24
 PUERTO USB\n
-Wire Notes Line
-	600  4550 8300 4550
 Wire Notes Line
 	8300 550  8300 4550
@@
 Wire Wire Line
 	1100 2950 600  2950
+Text Label 5350 5500 2    50   ~ 0
+SPI_CLK
+Text Label 5350 5350 2    50   ~ 0
+SPI_MOSI
+Wire Notes Line
+	550  550  550  4550
+Wire Notes Line
+	550  550  8300 550
+Wire Notes Line
+	550  4550 8300 4550
 Wire Bus Line
 	4450 5100 4450 5700
 Wire Bus Line
 	2150 5100 2150 5700
-Text Label 5350 5500 2    50   ~ 0
-SPI_CLK
-Text Label 5350 5350 2    50   ~ 0
-SPI_MOSI
 $EndSCHEMATC

Commit message: Add files via upload
Parts:
- C34, C36: footprint Resistor_SMD:R_0805_2012Metric_Pad1.15x1.40mm_HandSolder -> Resistor_SMD:R_0603_1608Metric_Pad1.05x0.95mm_HandSolder
- SW2: footprint libreria_proyecto_fp:LL3301NF065QG -> libreria_proyecto_fp:LL3301NF065QG-proy
Connections:
- net UART_RX renamed UART_O_RX
- net UART_TX renamed UART_O_TX
Changed lines of the file:
@@
 Wire Wire Line
 	2450 700  2450 1500
-Text Label 1400 2650 0    50   ~ 0
-RX_1
-Text Label 1400 2800 0    50   ~ 0
-TX_1
 Text Label 4550 5200 0    50   ~ 0
 SPI_fo0
@@
 F 0 "C34" H 6615 1096 50  0000 L CNN
 F 1 "22uF" H 6615 1005 50  0000 L CNN
-F 2 "Resistor_SMD:R_0805_2012Metric_Pad1.15x1.40mm_HandSolder" H 6538 900 50  0001 C CNN
+F 2 "Resistor_SMD:R_0603_1608Metric_Pad1.05x0.95mm_HandSolder" H 6538 900 50  0001 C CNN
 F 3 "~" H 6500 1050 50  0001 C CNN
 	1    6500 1050
@@
 F 0 "C36" H 7565 3596 50  0000 L CNN
 F 1 "22uF" H 7565 3505 50  0000 L CNN
-F 2 "Resistor_SMD:R_0805_2012Metric_Pad1.15x1.40mm_HandSolder" H 7488 3400 50  0001 C CNN
+F 2 "Resistor_SMD:R_0603_1608Metric_Pad1.05x0.95mm_HandSolder" H 7488 3400 50  0001 C CNN
 F 3 "~" H 7450 3550 50  0001 C CNN
 	1    7450 3550
@@
 F 0 "SW2" V 6496 3312 50  0000 R CNN
 F 1 "LL3301NF065QG-proy" V 6405 3312 50  0000 R CNN
-F 2 "libreria_proyecto_fp:LL3301NF065QG" H 6450 3800 50  0001 C CNN
+F 2 "libreria_proyecto_fp:LL3301NF065QG-proy" H 6450 3800 50  0001 C CNN
 F 3 "~" H 6450 3800 50  0001 C CNN
 	1    6450 3600
@@
 	1300 2800 1750 2800
 Text HLabel 1300 2800 0    50   Output ~ 0
-UART_TX
+UART_O_TX
 Text HLabel 1300 2650 0    50   Input ~ 0
-UART_RX
+UART_O_RX
 Wire Wire Line
 	1400 2950 1750 2950

Commit message: Add files via upload
Parts:
- added FB?: BLM18SG121TN1D-proy, Resistor_SMD:R_0603_1608Metric_Pad1.05x0.95mm_HandSolder, symbol try1-rescue:BLM18SG121TN1D-proy-proyecto_libreria
- D3: symbol Diode:BZX384C5V6-E3-08-proy -> try1-rescue:BZX384C5V6-E3-08-proy-Diode
- FB1: symbol proyecto_libreria:BLM18SG121TN1D-proy -> try1-rescue:BLM18SG121TN1D-proy-proyecto_libreria
- FL1: symbol proyecto_libreria:SRF2012A-900YA-proy -> try1-rescue:SRF2012A-900YA-proy-proyecto_libreria
- SW2: symbol proyecto_libreria:LL3301NF065QG-proy -> try1-rescue:LL3301NF065QG-proy-proyecto_libreria
- U5: symbol proyecto_libreria:Omega2-proy -> try1-rescue:Omega2-proy-proyecto_libreria
Connections:
- net GND: now also FB?.1; no longer J4.5 (Shield)
- new net: FB?.2, J4.5 (Shield)
Changed lines of the file:
@@
 $Descr User 8819 8110
 encoding utf-8
-Sheet 5 5
+Sheet 2 5
 Title ""
 Date ""
@@
 L power:GND #PWR0136
 U 1 1 5EEBD7D9
-P 5350 2100
+P 5400 2100
 AR Path="/5E81C316/5EEBD7D9" Ref="#PWR0136"  Part="1"
 AR Path="/5F32452B/5EEBD7D9" Ref="#PWR?"  Part="1"
-F 0 "#PWR0136" H 5350 1850 50  0001 C CNN
-F 1 "GND" H 5355 1927 50  0000 C CNN
-F 2 "" H 5350 2100 50  0001 C CNN
-F 3 "" H 5350 2100 50  0001 C CNN
-	1    5350 2100
+F 0 "#PWR0136" H 5400 1850 50  0001 C CNN
+F 1 "GND" H 5405 1927 50  0000 C CNN
+F 2 "" H 5400 2100 50  0001 C CNN
+F 3 "" H 5400 2100 50  0001 C CNN
+	1    5400 2100
 	1    0    0    -1
 $EndComp
 Wire Wire Line
 	5300 2000 5300 2050
-Wire Wire Line
-	5300 2050 5350 2050
-Wire Wire Line
-	5350 2050 5350 2100
-Wire Wire Line
-	5400 2000 5400 2050
-Wire Wire Line
-	5400 2050 5350 2050
-Connection ~ 5350 2050
 $Comp
 L Power_Protection:SP0502BAHT D4
@@
 	5700 850  6000 850
 $Comp
-L Diode:BZX384C5V6-E3-08-proy D3
+L try1-rescue:BZX384C5V6-E3-08-proy-Diode D3
 U 1 1 5EBA5BA1
 P 6000 1000
@@
 	6000 850  6500 850
 $Comp
-L proyecto_libreria:LL3301NF065QG-proy SW2
+L try1-rescue:LL3301NF065QG-proy-proyecto_libreria SW2
 U 1 1 5EBA7386
 P 6450 3600
@@
 $EndComp
 $Comp
-L proyecto_libreria:SRF2012A-900YA-proy FL1
+L try1-rescue:SRF2012A-900YA-proy-proyecto_libreria FL1
 U 1 1 5EBB9459
 P 7000 1600
@@
 $EndComp
 $Comp
-L proyecto_libreria:BLM18SG121TN1D-proy FB1
+L try1-rescue:BLM18SG121TN1D-proy-proyecto_libreria FB1
 U 1 1 5EBC1AC8
 P 7350 850
@@
 NoConn ~ 1750 2500
 $Comp
-L proyecto_libreria:Omega2-proy U5
+L try1-rescue:Omega2-proy-proyecto_libreria U5
 U 1 1 5EF04449
 P 2450 2850
@@
 Wire Notes Line
 	550  4550 8300 4550
+Wire Wire Line
+	5400 2000 5400 2100
+$Comp
+L try1-rescue:BLM18SG121TN1D-proy-proyecto_libreria FB?
+U 1 1 5ECF2138
+P 5300 2300
+AR Path="/5F3250E3/5ECF2138" Ref="FB?"  Part="1"
+AR Path="/5E81C316/5ECF2138" Ref="FB?"  Part="1"
+F 0 "FB?" H 5100 2550 50  0000 L CNN
+F 1 "BLM18SG121TN1D-proy" H 5100 2450 50  0000 L CNN
+F 2 "Resistor_SMD:R_0603_1608Metric_Pad1.05x0.95mm_HandSolder" H 5950 2400 50  0001 L CNN
+F 3 "https://www.murata.com/en-us/products/productdetail?partno=BLM18SG121TN1%23" H 5950 2300 50  0001 L CNN
+F 4 "Ferrite bead SMD 0603 120R 3A Murata Ferrite Bead (Chip Bead), 1.6 x 0.8 x 0.5mm (0603), 120 impedance at 100 MHz" H 5950 2200 50  0001 L CNN "Description"
+F 5 "0.75" H 5950 2100 50  0001 L CNN "Height"
+F 6 "Murata Electronics" H 5950 2000 50  0001 L CNN "Manufacturer_Name"
+F 7 "BLM18SG121TN1D" H 5950 1900 50  0001 L CNN "Manufacturer_Part_Number"
+F 8 "81-BLM18SG121TN1D" H 5950 1800 50  0001 L CNN "Mouser Part Number"
+F 9 "https://www.mouser.com/Search/Refine.aspx?Keyword=81-BLM18SG121TN1D" H 5950 1700 50  0001 L CNN "Mouser Price/Stock"
+F 10 "7241447P" H 5950 1600 50  0001 L CNN "RS Part Number"
+F 11 "http://uk.rs-online.com/web/p/products/7241447P" H 5950 1500 50  0001 L CNN "RS Price/Stock"
+	1    5300 2300
+	0    -1   -1   0
+$EndComp
 Wire Bus Line
 	4450 5100 4450 5700
 Wire Bus Line
 	2150 5100 2150 5700
+$Comp
+L power:GND #PWR?
+U 1 1 5ECFC1AF
+P 5300 2550
+AR Path="/5E81C316/5ECFC1AF" Ref="#PWR?"  Part="1"
+AR Path="/5F32452B/5ECFC1AF" Ref="#PWR?"  Part="1"
+F 0 "#PWR?" H 5300 2300 50  0001 C CNN
+F 1 "GND" H 5305 2377 50  0000 C CNN
+F 2 "" H 5300 2550 50  0001 C CNN
+F 3 "" H 5300 2550 50  0001 C CNN
+	1    5300 2550
+	0    -1   -1   0
+$EndComp
 $EndSCHEMATC
