File: kicad/Power_supply.sch (KiCad schematic (older format))
At the start: 27 parts, among them J5 USB_B_Micro, U10 ZLDO1117G33TA-proy, U6 ZLDO1117G12TA-proy, U7 ZLDO1117G25TA-proy, U8 ZLDO1117G33TA-proy, U9 ZLDO1117G33TA-proy

Commit message: Remove duplicated directory
Parts:
- removed FerriteBead3: BLM18SG121TN1D-proy, Inductor_SMD:L_0603_1608Metric_Pad1.05x0.95mm_HandSolder, symbol try1-rescue:BLM18SG121TN1D-proy-BLM18SG121TN1D
- added FB2, FB3, FB4, FB5, FB6: BLM18SG121TN1D-proy, Resistor_SMD:R_0603_1608Metric_Pad1.05x0.95mm_HandSolder, symbol proyecto_libreria:BLM18SG121TN1D-proy
- added H1, H2, H3, H4: MountingHole_Pad, MountingHole:MountingHole_2.5mm_Pad, symbol Mechanical:MountingHole_Pad
- C37, C38, C39, C43, C44, C45, C49, C50, C53, C54: footprint Capacitor_SMD:C_1206_3216Metric_Pad1.42x1.75mm_HandSolder -> Resistor_SMD:R_0805_2012Metric_Pad1.15x1.40mm_HandSolder
- C40, C41, C42, C47, C48, C51, C52: footprint Capacitor_SMD:C_0805_2012Metric_Pad1.15x1.40mm_HandSolder -> Resistor_SMD:R_0603_1608Metric_Pad1.05x0.95mm_HandSolder
- C46: footprint Capacitor_SMD:C_1206_3216Metric_Pad1.42x1.75mm_HandSolder -> Resistor_SMD:R_1206_3216Metric_Pad1.42x1.75mm_HandSolder
- R24: footprint Resistor_SMD:R_0805_2012Metric_Pad1.15x1.40mm_HandSolder -> Resistor_SMD:R_0603_1608Metric_Pad1.05x0.95mm_HandSolder
Connections:
- net +5V: now also FB2.2
- net GND: now also FB3.2, FB4.2, FB5.2, FB6.2
- net at J5.1 (VBUS): now also FB2.1
- new net: FB3.1, H1.1
- new net: FB4.1, H2.1
- new net: FB5.1, H3.1
- new net: FB6.1, H4.1
Other:
- note added: "Aimentacion FPGA\n\n"
- note added: "Aimentacion MICRO\n\n"
- note added: "Aimentacion OMEGA\n\n\n"
- note removed: "AL. FPGA\n\n"
- note removed: "AL. MICRO\n\n"
- note removed: "AL. OMEGA\n\n\n"

Commit message: Add files via upload
Parts:
- U10, U6, U7, U8, U9: footprint Package_TO_SOT_SMD:SOT-223-3_TabPin2 -> Package_TO_SOT_SMD:SOT-223
Changed lines of the file:
@@
 F 0 "U7" H 1550 4467 50  0000 C CNN
 F 1 "ZLDO1117G25TA-proy" H 1550 4376 50  0000 C CNN
-F 2 "Package_TO_SOT_SMD:SOT-223-3_TabPin2" H 350 3350 50  0001 C CIN
+F 2 "Package_TO_SOT_SMD:SOT-223" H 350 3350 50  0001 C CIN
 F 3 "https://www.infineon.com/dgdl/auips1051.pdf?fileId=5546d462533600a4015355a4710712fc" H 1550 4100 50  0001 C CNN
 	1    1550 4100
@@
 F 0 "U6" H 1550 3367 50  0000 C CNN
 F 1 "ZLDO1117G12TA-proy" H 1550 3276 50  0000 C CNN
-F 2 "Package_TO_SOT_SMD:SOT-223-3_TabPin2" H 350 2250 50  0001 C CIN
+F 2 "Package_TO_SOT_SMD:SOT-223" H 350 2250 50  0001 C CIN
 F 3 "https://www.infineon.com/dgdl/auips1051.pdf?fileId=5546d462533600a4015355a4710712fc" H 1550 3000 50  0001 C CNN
 	1    1550 3000
@@
 F 0 "U8" H 1550 5567 50  0000 C CNN
 F 1 "ZLDO1117G33TA-proy" H 1550 5476 50  0000 C CNN
-F 2 "Package_TO_SOT_SMD:SOT-223-3_TabPin2" H 350 4450 50  0001 C CIN
+F 2 "Package_TO_SOT_SMD:SOT-223" H 350 4450 50  0001 C CIN
 F 3 "https://www.infineon.com/dgdl/auips1051.pdf?fileId=5546d462533600a4015355a4710712fc" H 1550 5200 50  0001 C CNN
 	1    1550 5200
@@
 F 0 "U9" H 4300 3367 50  0000 C CNN
 F 1 "ZLDO1117G33TA-proy" H 4300 3276 50  0000 C CNN
-F 2 "Package_TO_SOT_SMD:SOT-223-3_TabPin2" H 3100 2250 50  0001 C CIN
+F 2 "Package_TO_SOT_SMD:SOT-223" H 3100 2250 50  0001 C CIN
 F 3 "https://www.infineon.com/dgdl/auips1051.pdf?fileId=5546d462533600a4015355a4710712fc" H 4300 3000 50  0001 C CNN
 	1    4300 3000
@@
 F 0 "U10" H 4300 4917 50  0000 C CNN
 F 1 "ZLDO1117G33TA-proy" H 4300 4826 50  0000 C CNN
-F 2 "Package_TO_SOT_SMD:SOT-223-3_TabPin2" H 3100 3800 50  0001 C CIN
+F 2 "Package_TO_SOT_SMD:SOT-223" H 3100 3800 50  0001 C CIN
 F 3 "https://www.infineon.com/dgdl/auips1051.pdf?fileId=5546d462533600a4015355a4710712fc" H 4300 4550 50  0001 C CNN
 	1    4300 4550

Commit message: Add files via upload
Parts:
- D5: footprint LED_SMD:LED_0805_2012Metric_Pad1.15x1.40mm_HandSolder -> LED_SMD:LED_0603_1608Metric_Pad1.05x0.95mm_HandSolder
Changed lines of the file:
@@
 F 0 "D5" V 4039 1383 50  0000 R CNN
 F 1 "LED" V 3948 1383 50  0000 R CNN
-F 2 "LED_SMD:LED_0805_2012Metric_Pad1.15x1.40mm_HandSolder" H 4000 1500 50  0001 C CNN
+F 2 "LED_SMD:LED_0603_1608Metric_Pad1.05x0.95mm_HandSolder" H 4000 1500 50  0001 C CNN
 F 3 "~" H 4000 1500 50  0001 C CNN
 	1    4000 1500

Commit message: Add files via upload
Parts:
- added FB9: BLM18SG121TN1D-proy, Resistor_SMD:R_0603_1608Metric_Pad1.05x0.95mm_HandSolder, symbol try1-rescue:BLM18SG121TN1D-proy-proyecto_libreria
- FB2, FB3, FB4, FB5, FB6: symbol proyecto_libreria:BLM18SG121TN1D-proy -> try1-rescue:BLM18SG121TN1D-proy-proyecto_libreria
- U10, U8, U9: symbol Regulator_Linear:ZLDO1117G33TA-proy -> try1-rescue:ZLDO1117G33TA-proy-Regulator_Linear
- U6: symbol Regulator_Linear:ZLDO1117G12TA-proy -> try1-rescue:ZLDO1117G12TA-proy-Regulator_Linear
- U7: symbol Regulator_Linear:ZLDO1117G25TA-proy -> try1-rescue:ZLDO1117G25TA-proy-Regulator_Linear
Connections:
- net GND: now also FB9.2; no longer J5.6 (Shield)
- new net GND_case: FB9.1, J5.6 (Shield)
Changed lines of the file:
@@
 $Descr User 9449 7520
 encoding utf-8
-Sheet 2 5
+Sheet 5 5
 Title ""
 Date ""
@@
 Wire Wire Line
 	1050 1950 1050 2000
-Wire Wire Line
-	1050 2000 1150 2000
-Wire Wire Line
-	1150 2000 1150 1950
-Wire Wire Line
-	1150 2100 1150 2000
-Connection ~ 1150 2000
 $Comp
 L Device:C C47
@@
 +1.2V_FPGA
 $Comp
-L Regulator_Linear:ZLDO1117G25TA-proy U7
+L try1-rescue:ZLDO1117G25TA-proy-Regulator_Linear U7
 U 1 1 5F398C7E
 P 1550 4100
@@
 $EndComp
 $Comp
-L Regulator_Linear:ZLDO1117G12TA-proy U6
+L try1-rescue:ZLDO1117G12TA-proy-Regulator_Linear U6
 U 1 1 5F39A05E
 P 1550 3000
@@
 $EndComp
 $Comp
-L Regulator_Linear:ZLDO1117G33TA-proy U8
+L try1-rescue:ZLDO1117G33TA-proy-Regulator_Linear U8
 U 1 1 5F39BD0D
 P 1550 5200
@@
 $EndComp
 $Comp
-L Regulator_Linear:ZLDO1117G33TA-proy U9
+L try1-rescue:ZLDO1117G33TA-proy-Regulator_Linear U9
 U 1 1 5F3E7978
 P 4300 3000
@@
 $EndComp
 $Comp
-L Regulator_Linear:ZLDO1117G33TA-proy U10
+L try1-rescue:ZLDO1117G33TA-proy-Regulator_Linear U10
 U 1 1 5F3E9E75
 P 4300 4550
@@
 	550  6250 3350 6250
 Wire Notes Line
-	8550 2450 8550 550
-Wire Notes Line
 	550  550  8550 550
-Wire Notes Line
-	550  2450 8550 2450
-$Comp
-L proyecto_libreria:BLM18SG121TN1D-proy FB2
+$Comp
+L try1-rescue:BLM18SG121TN1D-proy-proyecto_libreria FB2
 U 1 1 5EBB0508
 P 1950 1350
@@
 $EndComp
 $Comp
-L proyecto_libreria:BLM18SG121TN1D-proy FB3
+L try1-rescue:BLM18SG121TN1D-proy-proyecto_libreria FB3
 U 1 1 5EBB9E85
 P 4900 1500
@@
 $EndComp
 $Comp
-L proyecto_libreria:BLM18SG121TN1D-proy FB4
+L try1-rescue:BLM18SG121TN1D-proy-proyecto_libreria FB4
 U 1 1 5EBBC04B
 P 5800 1500
@@
 $EndComp
 $Comp
-L proyecto_libreria:BLM18SG121TN1D-proy FB5
+L try1-rescue:BLM18SG121TN1D-proy-proyecto_libreria FB5
 U 1 1 5EBBC5CD
 P 6700 1500
@@
 	7650 1750 7650 2000
 $Comp
-L proyecto_libreria:BLM18SG121TN1D-proy FB6
+L try1-rescue:BLM18SG121TN1D-proy-proyecto_libreria FB6
 U 1 1 5EBBD7F3
 P 7650 1500
@@
 	0    1    1    0
 $EndComp
+Wire Wire Line
+	1150 1950 1150 2100
+Text GLabel 1050 2000 0    50   Input ~ 0
+GND_case
+Text GLabel 6850 2500 0    50   Input ~ 0
+GND_case
+$Comp
+L try1-rescue:BLM18SG121TN1D-proy-proyecto_libreria FB9
+U 1 1 5ECCC61C
+P 7250 2500
+F 0 "FB9" H 7350 2650 50  0000 L CNN
+F 1 "BLM18SG121TN1D-proy" H 7295 2578 50  0000 L CNN
+F 2 "Resistor_SMD:R_0603_1608Metric_Pad1.05x0.95mm_HandSolder" H 7900 2600 50  0001 L CNN
+F 3 "https://www.murata.com/en-us/products/productdetail?partno=BLM18SG121TN1%23" H 7900 2500 50  0001 L CNN
+F 4 "Ferrite bead SMD 0603 120R 3A Murata Ferrite Bead (Chip Bead), 1.6 x 0.8 x 0.5mm (0603), 120 impedance at 100 MHz" H 7900 2400 50  0001 L CNN "Description"
+F 5 "0.75" H 7900 2300 50  0001 L CNN "Height"
+F 6 "Murata Electronics" H 7900 2200 50  0001 L CNN "Manufacturer_Name"
+F 7 "BLM18SG121TN1D" H 7900 2100 50  0001 L CNN "Manufacturer_Part_Number"
+F 8 "81-BLM18SG121TN1D" H 7900 2000 50  0001 L CNN "Mouser Part Number"
+F 9 "https://www.mouser.com/Search/Refine.aspx?Keyword=81-BLM18SG121TN1D" H 7900 1900 50  0001 L CNN "Mouser Price/Stock"
+F 10 "7241447P" H 7900 1800 50  0001 L CNN "RS Part Number"
+F 11 "http://uk.rs-online.com/web/p/products/7241447P" H 7900 1700 50  0001 L CNN "RS Price/Stock"
+	1    7250 2500
+	1    0    0    -1
+$EndComp
+$Comp
+L power:GND #PWR0168
+U 1 1 5ECCFD38
+P 7750 2550
+F 0 "#PWR0168" H 7750 2300 50  0001 C CNN
+F 1 "GND" H 7755 2377 50  0000 C CNN
+F 2 "" H 7750 2550 50  0001 C CNN
+F 3 "" H 7750 2550 50  0001 C CNN
+	1    7750 2550
+	1    0    0    -1
+$EndComp
+Wire Wire Line
+	7750 2500 7750 2550
+Wire Wire Line
+	7500 2500 7750 2500
+Wire Wire Line
+	7000 2500 6850 2500
+Wire Notes Line
+	6100 2450 550  2450
+Wire Notes Line
+	6100 2850 8550 2850
+Wire Notes Line
+	8550 550  8550 2850
 $EndSCHEMATC
