File: kicad/STM_32.sch (KiCad schematic (older format))
At the start: 12 parts, among them U4 STM32F100RBT6B-proy

Commit message: Remove duplicated directory
Parts:
- removed C31: 1uF, Capacitor_SMD:C_0805_2012Metric_Pad1.15x1.40mm_HandSolder, symbol Device:C
- removed FerriteBead1: 742792651-proy, Inductor_SMD:L_0603_1608Metric_Pad1.05x0.95mm_HandSolder, symbol try1-rescue:742792651-proy-742792651
- added FB7: BLM18SG121TN1D-proy, Resistor_SMD:R_0603_1608Metric_Pad1.05x0.95mm_HandSolder, symbol proyecto_libreria:BLM18SG121TN1D-proy
- C25, C26, C27, C28, C29, C30: footprint Capacitor_SMD:C_0805_2012Metric_Pad1.15x1.40mm_HandSolder -> Resistor_SMD:R_0603_1608Metric_Pad1.05x0.95mm_HandSolder
- R15, R16, R17: footprint Resistor_SMD:R_0805_2012Metric_Pad1.15x1.40mm_HandSolder -> Resistor_SMD:R_0603_1608Metric_Pad1.05x0.95mm_HandSolder
Connections:
- net +3.3V_micro: now also FB7.1; no longer U4.1 (VBAT)
- net GND: no longer C29.1, C30.1, U4.13 (VDDA)
- net JTAG_NRST: no longer names the net of U4.7 (NRST)
- net JTAG_TCK renamed JTAG1
- net JTAG_TDI renamed JTAG2
- net JTAG_TDO renamed JTAG3
- net JTAG_TMS renamed JTAG0
- net JTAG_TRST renamed JTAG4
- net SPI_CLK renamed SPI_mf1
- net SPI_MISO renamed SPI_mf2
- net SPI_MOSI renamed SPI_mf3
- net SPI_SS renamed SPI_mf0
- new net: C29.1, C30.1, FB7.2, U4.13 (VDDA)
- no-connect marks 0 -> 39
Other:
- moved on the sheet: C25, C26, C27, C28, C29, C30, R15, R16, R17, U4

Commit message: Add files via upload
Connections:
- net SPI_mf0: now also U4.22 (PA6/SPI1_MISO/ADC1_IN6/TIM3_CH1); no longer U4.20 (PA4/SPI1_NSS/DAC1_OUT/USART2_CK/ADC1_IN4)
- net SPI_mf1: now also U4.23 (PA7/SPI1_MOSI/ADC1_IN7/TIM3_CH2); no longer U4.21 (PA5/SPI1_SCK/DAC2_OUT/ADC1_IN5)
- net SPI_mf2: now also U4.21 (PA5/SPI1_SCK/DAC2_OUT/ADC1_IN5); no longer U4.22 (PA6/SPI1_MISO/ADC1_IN6/TIM3_CH1)
- net SPI_mf3: now also U4.20 (PA4/SPI1_NSS/DAC1_OUT/USART2_CK/ADC1_IN4); no longer U4.23 (PA7/SPI1_MOSI/ADC1_IN7/TIM3_CH2)
- net UART_M_TX: now reaches U4.51 (PC10/UART3_TX)
- net UART_M_RX: now reaches U4.52 (PC11/UART3_RX)
- net UART_RX: no longer names the net of U4.43 (PA10/USART1_RX/TIM1_CH3)
- net UART_TX: no longer names the net of U4.42 (PA9/USART1_TX/TIM1_CH2)
Changed lines of the file:
@@
 	4550 800  4100 800
 Connection ~ 4550 800
-Text HLabel 5650 3200 2    50   Input ~ 0
-UART_RX
-Text HLabel 5650 3100 2    50   Output ~ 0
-UART_TX
-Wire Wire Line
-	5650 3100 5450 3100
-Wire Wire Line
-	5450 3200 5650 3200
+Text HLabel 1450 5050 0    50   Input ~ 0
+UART_M_RX
+Text HLabel 1450 4950 0    50   Output ~ 0
+UART_M_TX
+Wire Wire Line
+	1450 4950 1650 4950
+Wire Wire Line
+	1650 5050 1450 5050
 $Comp
 L Device:R R17
@@
 Wire Bus Line
 	1350 6500 1450 6500
+Text Label 2650 6700 2    50   ~ 0
+SPI_micro_MISO
+Text Label 2650 6800 2    50   ~ 0
+SPI_micro_MOSI
+Text Label 2650 7000 2    50   ~ 0
+SPI_micro_SS
 Text Label 2650 6900 2    50   ~ 0
-SPI_micro_MISO
-Text Label 2650 7000 2    50   ~ 0
-SPI_micro_MOSI
-Text Label 2650 6700 2    50   ~ 0
-SPI_micro_SS
-Text Label 2650 6800 2    50   ~ 0
 SPI_micro_CLK
 Wire Wire Line
+	1550 6700 2650 6700
+Wire Wire Line
+	1550 6800 2650 6800
+Wire Wire Line
+	1550 7000 2650 7000
+Wire Wire Line
 	1550 6900 2650 6900
-Wire Wire Line
-	1550 7000 2650 7000
-Wire Wire Line
-	1550 6700 2650 6700
-Wire Wire Line
-	1550 6800 2650 6800
 Wire Wire Line
 	5450 4550 6000 4550
@@
 NoConn ~ 1650 5250
 NoConn ~ 1650 5150
-NoConn ~ 1650 5050
-NoConn ~ 1650 4950
 NoConn ~ 1650 4850
 NoConn ~ 1650 4750
@@
 Wire Wire Line
 	5450 4350 6550 4350
+NoConn ~ 5450 3100
+NoConn ~ 5450 3200
 Wire Bus Line
 	3350 6500 3350 6700

Commit message: Add files via upload
Parts:
- added FB8: BLM18SG121TN1D-proy, Resistor_SMD:R_0603_1608Metric_Pad1.05x0.95mm_HandSolder, symbol try1-rescue:BLM18SG121TN1D-proy-proyecto_libreria
- FB7: symbol proyecto_libreria:BLM18SG121TN1D-proy -> try1-rescue:BLM18SG121TN1D-proy-proyecto_libreria
- U4: symbol MCU_ST_STM32F1:STM32F100RBT6B-proy -> try1-rescue:STM32F100RBT6B-proy-MCU_ST_STM32F1
Connections:
- net GND: now also FB8.1; no longer U4.12 (VSSA)
- new net: FB8.2, U4.12 (VSSA)
Changed lines of the file:
@@
 $Descr A4 11693 8268
 encoding utf-8
-Sheet 3 5
+Sheet 4 5
 Title ""
 Date ""
@@
 Wire Wire Line
 	5550 7100 6650 7100
-$Comp
-L proyecto_libreria:BLM18SG121TN1D-proy FB7
-U 1 1 5EBA01FD
-P 3700 1100
-F 0 "FB7" H 3700 1315 50  0000 C CNN
-F 1 "BLM18SG121TN1D-proy" H 3700 1224 50  0000 C CNN
-F 2 "Resistor_SMD:R_0603_1608Metric_Pad1.05x0.95mm_HandSolder" H 4350 1200 50  0001 L CNN
-F 3 "https://www.murata.com/en-us/products/productdetail?partno=BLM18SG121TN1%23" H 4350 1100 50  0001 L CNN
-F 4 "Ferrite bead SMD 0603 120R 3A Murata Ferrite Bead (Chip Bead), 1.6 x 0.8 x 0.5mm (0603), 120 impedance at 100 MHz" H 4350 1000 50  0001 L CNN "Description"
-F 5 "0.75" H 4350 900 50  0001 L CNN "Height"
-F 6 "Murata Electronics" H 4350 800 50  0001 L CNN "Manufacturer_Name"
-F 7 "BLM18SG121TN1D" H 4350 700 50  0001 L CNN "Manufacturer_Part_Number"
-F 8 "81-BLM18SG121TN1D" H 4350 600 50  0001 L CNN "Mouser Part Number"
-F 9 "https://www.mouser.com/Search/Refine.aspx?Keyword=81-BLM18SG121TN1D" H 4350 500 50  0001 L CNN "Mouser Price/Stock"
-F 10 "7241447P" H 4350 400 50  0001 L CNN "RS Part Number"
-F 11 "http://uk.rs-online.com/web/p/products/7241447P" H 4350 300 50  0001 L CNN "RS Price/Stock"
-	1    3700 1100
-	1    0    0    -1
-$EndComp
 NoConn ~ 1650 3000
 NoConn ~ 1650 3100
@@
 NoConn ~ 5450 2300
 NoConn ~ 5450 2200
-Wire Wire Line
-	3700 6150 3600 6150
-Connection ~ 3600 6150
-Wire Wire Line
-	3500 1550 3600 1550
-Connection ~ 3500 1550
-Wire Wire Line
-	3500 6150 3600 6150
-Connection ~ 3500 6150
-Wire Wire Line
-	3300 1550 3400 1550
-Wire Wire Line
-	3400 1550 3500 1550
-Connection ~ 3400 1550
-Wire Wire Line
-	3300 6150 3400 6150
-Wire Wire Line
-	3400 6150 3500 6150
-Connection ~ 3400 6150
-Connection ~ 3300 1550
-Connection ~ 3300 6150
-$Comp
-L MCU_ST_STM32F1:STM32F100RBT6B-proy U4
-U 1 1 5EA2851A
-P 3500 4250
-F 0 "U4" H 2000 6800 50  0000 C CNN
-F 1 "STM32F100RBT6B-proy" H 2400 6700 50  0000 C CNN
-F 2 "Package_QFP:LQFP-64_10x10mm_P0.5mm" H 1950 2950 50  0001 R CNN
-F 3 "http://www.st.com/st-web-ui/static/active/en/resource/technical/document/datasheet/CD00251732.pdf" H 3300 4500 50  0001 C CNN
-	1    3500 4250
-	1    0    0    -1
-$EndComp
 NoConn ~ 5050 1550
 Wire Wire Line
@@
 NoConn ~ 5450 3100
 NoConn ~ 5450 3200
+Wire Wire Line
+	3500 1550 3600 1550
+Connection ~ 3500 1550
+Wire Wire Line
+	3500 6150 3600 6150
+Connection ~ 3500 6150
+Wire Wire Line
+	3400 1550 3500 1550
+Wire Wire Line
+	3300 1550 3400 1550
+Connection ~ 3400 1550
+Wire Wire Line
+	3400 6150 3500 6150
+Wire Wire Line
+	3300 6150 3400 6150
+Connection ~ 3400 6150
+Connection ~ 3300 1550
+Connection ~ 3300 6150
+$Comp
+L try1-rescue:STM32F100RBT6B-proy-MCU_ST_STM32F1 U4
+U 1 1 5EA2851A
+P 3500 4250
+F 0 "U4" H 2000 6800 50  0000 C CNN
+F 1 "STM32F100RBT6B-proy" H 2400 6700 50  0000 C CNN
+F 2 "Package_QFP:LQFP-64_10x10mm_P0.5mm" H 1950 2950 50  0001 R CNN
+F 3 "http://www.st.com/st-web-ui/static/active/en/resource/technical/document/datasheet/CD00251732.pdf" H 3300 4500 50  0001 C CNN
+	1    3500 4250
+	1    0    0    -1
+$EndComp
+$Comp
+L try1-rescue:BLM18SG121TN1D-proy-proyecto_libreria FB7
+U 1 1 5EBA01FD
+P 3700 1100
+F 0 "FB7" H 3700 1315 50  0000 C CNN
+F 1 "BLM18SG121TN1D-proy" H 3700 1224 50  0000 C CNN
+F 2 "Resistor_SMD:R_0603_1608Metric_Pad1.05x0.95mm_HandSolder" H 4350 1200 50  0001 L CNN
+F 3 "https://www.murata.com/en-us/products/productdetail?partno=BLM18SG121TN1%23" H 4350 1100 50  0001 L CNN
+F 4 "Ferrite bead SMD 0603 120R 3A Murata Ferrite Bead (Chip Bead), 1.6 x 0.8 x 0.5mm (0603), 120 impedance at 100 MHz" H 4350 1000 50  0001 L CNN "Description"
+F 5 "0.75" H 4350 900 50  0001 L CNN "Height"
+F 6 "Murata Electronics" H 4350 800 50  0001 L CNN "Manufacturer_Name"
+F 7 "BLM18SG121TN1D" H 4350 700 50  0001 L CNN "Manufacturer_Part_Number"
+F 8 "81-BLM18SG121TN1D" H 4350 600 50  0001 L CNN "Mouser Part Number"
+F 9 "https://www.mouser.com/Search/Refine.aspx?Keyword=81-BLM18SG121TN1D" H 4350 500 50  0001 L CNN "Mouser Price/Stock"
+F 10 "7241447P" H 4350 400 50  0001 L CNN "RS Part Number"
+F 11 "http://uk.rs-online.com/web/p/products/7241447P" H 4350 300 50  0001 L CNN "RS Price/Stock"
+	1    3700 1100
+	1    0    0    -1
+$EndComp
+$Comp
+L try1-rescue:BLM18SG121TN1D-proy-proyecto_libreria FB8
+U 1 1 5ECD6661
+P 4050 6150
+F 0 "FB8" H 4050 6365 50  0000 C CNN
+F 1 "BLM18SG121TN1D-proy" H 4050 6274 50  0000 C CNN
+F 2 "Resistor_SMD:R_0603_1608Metric_Pad1.05x0.95mm_HandSolder" H 4700 6250 50  0001 L CNN
+F 3 "https://www.murata.com/en-us/products/productdetail?partno=BLM18SG121TN1%23" H 4700 6150 50  0001 L CNN
+F 4 "Ferrite bead SMD 0603 120R 3A Murata Ferrite Bead (Chip Bead), 1.6 x 0.8 x 0.5mm (0603), 120 impedance at 100 MHz" H 4700 6050 50  0001 L CNN "Description"
+F 5 "0.75" H 4700 5950 50  0001 L CNN "Height"
+F 6 "Murata Electronics" H 4700 5850 50  0001 L CNN "Manufacturer_Name"
+F 7 "BLM18SG121TN1D" H 4700 5750 50  0001 L CNN "Manufacturer_Part_Number"
+F 8 "81-BLM18SG121TN1D" H 4700 5650 50  0001 L CNN "Mouser Part Number"
+F 9 "https://www.mouser.com/Search/Refine.aspx?Keyword=81-BLM18SG121TN1D" H 4700 5550 50  0001 L CNN "Mouser Price/Stock"
+F 10 "7241447P" H 4700 5450 50  0001 L CNN "RS Part Number"
+F 11 "http://uk.rs-online.com/web/p/products/7241447P" H 4700 5350 50  0001 L CNN "RS Price/Stock"
+	1    4050 6150
+	-1   0    0    1
+$EndComp
+$Comp
+L power:GND #PWR0111
+U 1 1 5ECD825F
+P 4300 6150
+F 0 "#PWR0111" H 4300 5900 50  0001 C CNN
+F 1 "GND" H 4305 5977 50  0000 C CNN
+F 2 "" H 4300 6150 50  0001 C CNN
+F 3 "" H 4300 6150 50  0001 C CNN
+	1    4300 6150
+	0    -1   -1   0
+$EndComp
+Wire Wire Line
+	3800 6150 3700 6150
 Wire Bus Line
 	3350 6500 3350 6700
 Wire Bus Line
+	5450 6500 5450 7000
+Wire Bus Line
 	1450 6500 1450 6900
-Wire Bus Line
-	5450 6500 5450 7000
 $EndSCHEMATC
