File: kicad/try1.sch (KiCad schematic (older format))
At the start: 0 parts

Commit message: Remove duplicated directory
Changed lines of the file:
@@
 Wire Bus Line
 	2950 3900 2400 3900
-$Sheet
-S 3200 950  1450 1300
-U 5E81C2A4
-F0 "FPGA_ICE40UP5K" 50
-F1 "FPGA_ICE40UP5K.sch" 50
-F2 "I2C_fpga[1..0]" B L 3200 1450 50
-F3 "SPI_fpga_omega[4..0]" B L 3200 2050 50
-F4 "SPI_fpga[3..0]" B L 3200 1250 50
-$EndSheet
-$Sheet
-S 1050 950  1350 1300
-U 5E81C399
-F0 "STM_32" 50
-F1 "STM_32.sch" 50
-F2 "BOOT0" I L 1050 1500 50
-F3 "UART_RX" I R 2400 2150 50
-F4 "UART_TX" O R 2400 2050 50
-F5 "BOOT1" I L 1050 1650 50
-F6 "SPI_micro[3..0]" B R 2400 1250 50
-F7 "I2C_micro[1..0]" B R 2400 1450 50
-F8 "JATG_micro[5..0]" B R 2400 1950 50
-$EndSheet
-$Sheet
-S 1050 2750 1350 1250
-U 5E81C316
-F0 "Onion_2" 50
-F1 "Onion_2.sch" 50
-F2 "JTAG[5..0]" B R 2400 3200 50
-F3 "I2C_omega[1..0]" B R 2400 3600 50
-F4 "BOOT1" O L 1050 3050 50
-F5 "UART_RX" I R 2400 2950 50
-F6 "UART_TX" O R 2400 2850 50
-F7 "BOOT0" O L 1050 3200 50
-F8 "SPI_omega_fpga[4..0]" B R 2400 3900 50
-$EndSheet
 Wire Wire Line
 	1050 3050 1000 3050
@@
 F1 "Power_supply.sch" 50
 $EndSheet
+$Sheet
+S 1050 950  1350 1300
+U 5E81C399
+F0 "STM_32" 50
+F1 "STM_32.sch" 50
+F2 "BOOT0" I L 1050 1500 50
+F3 "UART_RX" I R 2400 2150 50
+F4 "UART_TX" O R 2400 2050 50
+F5 "BOOT1" I L 1050 1650 50
+F6 "SPI_mf[3..0]" B R 2400 1250 50
+F7 "I2C_all[1..0]" B R 2400 1450 50
+F8 "JTAG[4..0]" B R 2400 1950 50
+$EndSheet
+$Sheet
+S 3200 950  1450 1300
+U 5E81C2A4
+F0 "FPGA_ICE40UP5K" 50
+F1 "FPGA_ICE40UP5K.sch" 50
+F2 "SPI_fo[4..0]" B L 3200 2050 50
+F3 "I2C_all[1..0]" B L 3200 1450 50
+F4 "SPI_mf[3..0]" B L 3200 1250 50
+$EndSheet
+$Sheet
+S 1050 2750 1350 1250
+U 5E81C316
+F0 "Onion_2" 50
+F1 "Onion_2.sch" 50
+F2 "BOOT1" O L 1050 3050 50
+F3 "UART_RX" I R 2400 2950 50
+F4 "UART_TX" O R 2400 2850 50
+F5 "BOOT0" O L 1050 3200 50
+F6 "I2C_all[1..0]" B R 2400 3600 50
+F7 "JTAG[4..0]" B R 2400 3200 50
+F8 "SPI_fo[4..0]" B R 2400 3900 50
+$EndSheet
 $EndSCHEMATC

Commit message: Add files via upload
Changed lines of the file:
@@
 F1 "STM_32.sch" 50
 F2 "BOOT0" I L 1050 1500 50
-F3 "UART_RX" I R 2400 2150 50
-F4 "UART_TX" O R 2400 2050 50
-F5 "BOOT1" I L 1050 1650 50
-F6 "SPI_mf[3..0]" B R 2400 1250 50
-F7 "I2C_all[1..0]" B R 2400 1450 50
-F8 "JTAG[4..0]" B R 2400 1950 50
+F3 "BOOT1" I L 1050 1650 50
+F4 "SPI_mf[3..0]" B R 2400 1250 50
+F5 "I2C_all[1..0]" B R 2400 1450 50
+F6 "JTAG[4..0]" B R 2400 1950 50
+F7 "UART_M_RX" I R 2400 2150 50
+F8 "UART_M_TX" O R 2400 2050 50
 $EndSheet
 $Sheet
@@
 F1 "Onion_2.sch" 50
 F2 "BOOT1" O L 1050 3050 50
-F3 "UART_RX" I R 2400 2950 50
-F4 "UART_TX" O R 2400 2850 50
-F5 "BOOT0" O L 1050 3200 50
-F6 "I2C_all[1..0]" B R 2400 3600 50
-F7 "JTAG[4..0]" B R 2400 3200 50
-F8 "SPI_fo[4..0]" B R 2400 3900 50
+F3 "BOOT0" O L 1050 3200 50
+F4 "I2C_all[1..0]" B R 2400 3600 50
+F5 "JTAG[4..0]" B R 2400 3200 50
+F6 "SPI_fo[4..0]" B R 2400 3900 50
+F7 "UART_O_TX" O R 2400 2850 50
+F8 "UART_O_RX" I R 2400 2950 50
 $EndSheet
 $EndSCHEMATC
